Commit message: Integrate ella gripper + workspace MoveIt planning config
Long-standing local workspace adaptations, committed for the record:
- tm5x-900 xacro: include ella_gripper.xacro; restrict joint_2 to
  +/-80 deg; default color/format params
- srdf: ella gripper link collision exclusions; home config joints
  set to the workspace home (j2 -0.8, j3 1.8, j4 -4.13, j5 -1.57)
- joint_limits: velocity/acceleration scaling 0.1 -> 1.0, enable
  acceleration limits (10.5 rad/s^2)
- ompl/chomp planning tweaks
- tm5x-900_moveit.launch.py (real-robot variant): add ella_controller
  tcp_communication + test_angles nodes; tm5-900 launch touch-up

Co-Authored-By: Claude Opus 4.8 <noreply@anthropic.com>

File: tm_description/xacro/macro.tm5x-900-nominal.urdf.xacro (robot description, xacro)
@@ -2,7 +2,8 @@
 <robot xmlns:xacro="http://www.ros.org/wiki/xacro">
   <xacro:include filename="$(find tm_description)/xacro/macro.inertial.xacro" />
-  <xacro:macro name="tm5x-900" params="ns prefix color format
+  <xacro:include filename="$(find ella_gripper_description)/urdf/ella_gripper.xacro" />
+  <xacro:macro name="tm5x-900" params="ns prefix color:=none format:=obj
     joint_1_lower_limit:=${radians(-360)}    joint_1_upper_limit:=${radians(360)}
-    joint_2_lower_limit:=${radians(-360)}    joint_2_upper_limit:=${radians(360)}
+    joint_2_lower_limit:=${radians(-80)}    joint_2_upper_limit:=${radians(80)}
     joint_3_lower_limit:=${radians(-155)}    joint_3_upper_limit:=${radians(155)}
     joint_4_lower_limit:=${radians(-360)}    joint_4_upper_limit:=${radians(360)}
@@ -23,18 +24,18 @@
     safety_limits:=false safety_pos_margin:=0.15
     safety_k_position:=20">
-    <xacro:property name="damping_factor" value="0.000"/>
-    <xacro:property name="d1" value="${damping_factor*0.1}"/>
-    <xacro:property name="d2" value="${damping_factor*0.1}"/>
-    <xacro:property name="d3" value="${damping_factor*0.1}"/>
-    <xacro:property name="d4" value="${damping_factor*0.1}"/>
-    <xacro:property name="d5" value="${damping_factor*0.1}"/>
-    <xacro:property name="d6" value="${damping_factor*0.1}"/>
-    <xacro:property name="friction_factor" value="0.000"/>
-    <xacro:property name="f1" value="${friction_factor*0.1}"/>
-    <xacro:property name="f2" value="${friction_factor*0.1}"/>
-    <xacro:property name="f3" value="${friction_factor*0.1}"/>
-    <xacro:property name="f4" value="${friction_factor*0.1}"/>
-    <xacro:property name="f5" value="${friction_factor*0.1}"/>
-    <xacro:property name="f6" value="${friction_factor*0.1}"/>
+   <xacro:property name="damping_factor" value="0.000"/>
+   <xacro:property name="d1" value="${damping_factor*0.1}"/>
+   <xacro:property name="d2" value="${damping_factor*0.1}"/>
+   <xacro:property name="d3" value="${damping_factor*0.1}"/>
+   <xacro:property name="d4" value="${damping_factor*0.1}"/>
+   <xacro:property name="d5" value="${damping_factor*0.1}"/>
+   <xacro:property name="d6" value="${damping_factor*0.1}"/>
+   <xacro:property name="friction_factor" value="0.000"/>
+   <xacro:property name="f1" value="${friction_factor*0.1}"/>
+   <xacro:property name="f2" value="${friction_factor*0.1}"/>
+   <xacro:property name="f3" value="${friction_factor*0.1}"/>
+   <xacro:property name="f4" value="${friction_factor*0.1}"/>
+   <xacro:property name="f5" value="${friction_factor*0.1}"/>
+   <xacro:property name="f6" value="${friction_factor*0.1}"/>
     <!-- Inertia parameters -->
     <xacro:property name="mass_0" value="1.000" />
@@ -64,18 +65,4 @@
     <xacro:property name="izz_5" value="${2643.21*unit_factor}" />
     <xacro:property name="izz_6" value="${286.595*unit_factor}" />
-    <xacro:property name="specified_color_arms" default="false" />
-    <xacro:property name="prefix_monochrome_command" default="true" />
-    <!-- If other applications conflict with the color definition of URDF, try disable_prefix_color to close it -->
-    <xacro:property name="disable_prefix_color" default="false" />
-    <xacro:if value="${disable_prefix_color}">
-      <prefix_monochrome_command value="false"/>
-    </xacro:if>
-    <xacro:if value="${format == 'stl'}">
-      <specified_color_arms value="true"/>
-      <prefix_monochrome_command value="false"/>
-    </xacro:if>
-    <xacro:if value="${prefix_monochrome_command}">
-      <xacro:tm_materials/>
-    </xacro:if>
 <!--LinkDescription-->
   <link name="${prefix}link_0">
@@ -84,10 +71,5 @@
         <mesh filename="package://tm_description/meshes/tm5-900/visual/tm5-base.${format}" />
       </geometry>
-      <xacro:if value="${specified_color_arms}">
-        <xacro:tm_material_whitegraphite />
-      </xacro:if>
-      <xacro:if value="${prefix_monochrome_command}">
-        <material name="${color}" />
-      </xacro:if>
+      <material name="${color}" />
     </visual>
     <collision>
@@ -118,10 +100,5 @@
         <mesh filename="package://tm_description/meshes/tm5-900/visual/tmr_400w_01.${format}" />
       </geometry>
-      <xacro:if value="${specified_color_arms}">
-        <xacro:tm_material_darkolive />
-      </xacro:if>
-      <xacro:if value="${prefix_monochrome_command}">
-        <material name="${color}" />
-      </xacro:if>
+      <material name="${color}" />
     </visual>
     <collision>
@@ -153,10 +130,5 @@
         <mesh filename="package://tm_description/meshes/tm5-900/visual/tm5-900_arm1.${format}" />
       </geometry>
-      <xacro:if value="${specified_color_arms}">
-        <xacro:tm_material_darkolive />
-      </xacro:if>
-      <xacro:if value="${prefix_monochrome_command}">
-        <material name="${color}" />
-      </xacro:if>
+      <material name="${color}" />
     </visual>
     <collision>
@@ -188,10 +160,5 @@
         <mesh filename="package://tm_description/meshes/tm5-900/visual/tm5-900_arm2.${format}" />
       </geometry>
-      <xacro:if value="${specified_color_arms}">
-        <xacro:tm_material_gold />
-      </xacro:if>
-      <xacro:if value="${prefix_monochrome_command}">
-        <material name="${color}" />
-      </xacro:if>
+      <material name="${color}" />
     </visual>
     <collision>
@@ -223,10 +190,5 @@
         <mesh filename="package://tm_description/meshes/tm5-900/visual/tmr_100w_01.${format}" />
       </geometry>
-      <xacro:if value="${specified_color_arms}">
-        <xacro:tm_material_darkolive />
-      </xacro:if>
-      <xacro:if value="${prefix_monochrome_command}">
-        <material name="${color}" />
-      </xacro:if>
+      <material name="${color}" />
     </visual>
     <collision>
@@ -258,10 +220,5 @@
         <mesh filename="package://tm_description/meshes/tm5-900/visual/tmr_100w_02.${format}" />
       </geometry>
-      <xacro:if value="${specified_color_arms}">
-        <xacro:tm_material_darkolive />
-      </xacro:if>
-      <xacro:if value="${prefix_monochrome_command}">
-        <material name="${color}" />
-      </xacro:if>
+      <material name="${color}" />
     </visual>
     <collision>
@@ -293,10 +250,5 @@
         <mesh filename="package://tm_description/meshes/tm5-900/visual/tmr_iox.${format}" />
       </geometry>
-      <xacro:if value="${specified_color_arms}">
-        <xacro:tm_material_purewhite />
-      </xacro:if>
-      <xacro:if value="${prefix_monochrome_command}">
-        <material name="${color}" />
-      </xacro:if>
+      <material name="${color}" />
     </visual>
     <collision>
@@ -311,4 +263,10 @@
     </inertial>
   </link>
+  <link name="world"/>
+  <joint name="world_to_base" type="fixed">
+    <parent link="world"/>
+    <child link="base"/>
+    <origin xyz="0 0 0" rpy="0 0 0"/>
+  </joint>
   <link name="${prefix}base" />
   <joint name="${prefix}base_fixed_joint" type="fixed">
@@ -321,7 +279,9 @@
     <parent link="${prefix}link_6" />
     <child link="${prefix}flange" />
-    <origin rpy="0.000000 0.000000 0.000000" xyz="0.000000 0.000000 0.000000" />
+    <origin rpy="0.000000 0.000000 0.000000" xyz="0.00000 0.000000 0.230000" />
   </joint>
 <!--LinkDescription-->
+<!-- Attach Ella Gripper at TM flange -->
+<xacro:ella_gripper parent_link="${prefix}link_6"/>
   </xacro:macro>
 </robot>
